File: PCB/edge-lord-2000.brd (EAGLE design)
At the start: 52 x 100 mm, 40 parts, among them Q1 SI2302CDS, Q2 SI2302CDS, Q3 SI2302CDS, Q4 SI2302CDS, Q5 ON Semi NTS4173P, Q6 2N7002

Commit message: PWR switch was backward. Updated 3D model for fusion.
Connections:
- net N$1 renamed EN
- net GND: now also PWR.3; no longer PWR.1
Changed lines of the file:
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@@
 </layers>
 <board>
-<fusionsync huburn="a.cGVyc29uYWw6dWUyYmRlZGJl" projecturn="a.cGVyc29uYWw6dWUyYmRlZGJlIzIwMTcwMzI1Njg5MjEzMDY" f3durn="urn:adsk.wipprod:dm.lineage:VkQONFKbSQmlTrznlbgTTQ" pcbguid="" lastpulledtime="" lastsyncedchangeguid="" latestrevisionid="58f3acec-7e41-46b0-b4b5-7cada9a63452" lastsyncedrevisionid="58f3acec-7e41-46b0-b4b5-7cada9a63452" lastboardhashguid="8f786de1-8546-1301-88f5-f3cb95fc9794" lastpushedtime="2021-12-28T23:39:31Z" linktopcb3d="true"/>
+<fusionsync huburn="a.cGVyc29uYWw6dWUyYmRlZGJl" projecturn="a.cGVyc29uYWw6dWUyYmRlZGJlIzIwMTgwNTA0MTMwNTkwMzU2" f3durn="urn:adsk.wipprod:dm.lineage:Owe0uUw4Qyar69ouMgCf0w" pcbguid="51dd95b6-2379-4a06-a81f-2d97e1af3568" lastpulledtime="" lastsyncedchangeguid="" latestrevisionid="f083e808-b7ae-4063-8117-84aeecfaca73" lastsyncedrevisionid="f083e808-b7ae-4063-8117-84aeecfaca73" lastboardhashguid="edf6f39f-40e3-2f56-e119-07d7723e7346" lastpushedtime="2022-04-19T22:39:49Z" linktopcb3d="true"/>
 <plain>
 <wire x1="4" y1="0" x2="48" y2="0" width="0" layer="20"/>
@@
 </elements>
 <signals>
-<signal name="N$1">
+<signal name="EN">
 <contactref element="HUZZAH" pad="EN"/>
 <contactref element="PWR" pad="2"/>
@@
 <contactref element="RGB3" pad="2"/>
 <contactref element="R7" pad="1"/>
-<contactref element="PWR" pad="1"/>
 <contactref element="C12" pad="2"/>
 <contactref element="C13" pad="2"/>
@@
 <via x="25.9" y="20.3" extent="1-16" drill="0.35"/>
 <via x="34.6" y="20" extent="1-16" drill="0.35"/>
+<contactref element="PWR" pad="3"/>
 </signal>
 <signal name="+4.1V">

Commit message: PCB Rev.A tweaks.
Parts:
- R4: value XXX -> 330
Changed lines of the file:
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@@
 </layers>
 <board>
-<fusionsync huburn="a.cGVyc29uYWw6dWUyYmRlZGJl" projecturn="a.cGVyc29uYWw6dWUyYmRlZGJlIzIwMTgwNTA0MTMwNTkwMzU2" f3durn="urn:adsk.wipprod:dm.lineage:Owe0uUw4Qyar69ouMgCf0w" pcbguid="51dd95b6-2379-4a06-a81f-2d97e1af3568" lastpulledtime="" lastsyncedchangeguid="" latestrevisionid="f083e808-b7ae-4063-8117-84aeecfaca73" lastsyncedrevisionid="f083e808-b7ae-4063-8117-84aeecfaca73" lastboardhashguid="edf6f39f-40e3-2f56-e119-07d7723e7346" lastpushedtime="2022-04-19T22:39:49Z" linktopcb3d="true"/>
+<fusionsync huburn="a.cGVyc29uYWw6dWUyYmRlZGJl" projecturn="a.cGVyc29uYWw6dWUyYmRlZGJlIzIwMTgwNTA0MTMwNTkwMzU2" f3durn="urn:adsk.wipprod:dm.lineage:Owe0uUw4Qyar69ouMgCf0w" pcbguid="" lastpulledtime="" lastsyncedchangeguid="" latestrevisionid="f083e808-b7ae-4063-8117-84aeecfaca73" lastsyncedrevisionid="f083e808-b7ae-4063-8117-84aeecfaca73" lastboardhashguid="edf6f39f-40e3-2f56-e119-07d7723e7346" lastpushedtime="2022-04-19T22:39:49Z" linktopcb3d="true"/>
 <plain>
 <wire x1="4" y1="0" x2="48" y2="0" width="0" layer="20"/>
@@
 <attribute name="VALUE" value="XXX" x="16.9" y="59.1" size="0.2" layer="27" rot="R90" align="center"/>
 </element>
-<element name="R4" library="rlc" library_urn="urn:adsk.eagle:library:4192893" package="0603-RES" package3d_urn="urn:adsk.eagle:package:4193040/2" value="XXX" x="27.2" y="59.1" smashed="yes" rot="R270">
+<element name="R4" library="rlc" library_urn="urn:adsk.eagle:library:4192893" package="0603-RES" package3d_urn="urn:adsk.eagle:package:4193040/2" value="330" x="27.2" y="59.1" smashed="yes" rot="R270">
 <attribute name="COST01" value="0.10" x="27.2" y="59.1" size="1.778" layer="27" rot="R270" display="off"/>
 <attribute name="COST10" value="0.05" x="27.2" y="59.1" size="1.778" layer="27" rot="R270" display="off"/>

Commit message: More notes in PCB. Update Huzzah symbol.
Parts:
- C11, C12, C13: value 1uF -> ??uF
- C6, C7, C8, C9: value 0.1uF -> ??uF
- HUZZAH: value (none) -> Huzzah32
